Commit message: Update marker positions to have greater assymmetry

File: urdf/anymal_vicon_markers.urdf.xacro (robot description, xacro)
@@ -9,5 +9,5 @@
   <xacro:include filename="$(find anymal_boxy_description)/urdf/anymal.urdf.xacro"/>
   <xacro:property name="vicon_marker_size" value="0.007"/>
-  <xacro:property name="standoff_height" value="0.030"/>
+  <xacro:property name="standoff_height" value="0.020"/>
   <xacro:property name="standoff_radius" value="0.002"/>
   <link name="vicon/marker1">
@@ -29,5 +29,5 @@
     <parent link="base"/>
     <child link="vicon/marker1"/>
-    <origin rpy="0 0 ${pi/2}" xyz="0.196 -0.1 0.23"/>
+    <origin rpy="0 0 ${pi/2}" xyz="0.196 -0.099 0.22"/>
   </joint>
   <link name="vicon/marker2">
@@ -49,5 +49,5 @@
     <parent link="base"/>
     <child link="vicon/marker2"/>
-    <origin rpy="0 0 ${pi/2}" xyz="0.196 0.1 0.23"/>
+    <origin rpy="0 0 ${pi/2}" xyz="0.126 0.099 0.22"/>
   </joint>
   <link name="vicon/marker3">
@@ -69,5 +69,5 @@
     <parent link="base"/>
     <child link="vicon/marker3"/>
-    <origin rpy="0 0 ${pi/2}" xyz="-0.125 -0.1 0.23"/>
+    <origin rpy="0 0 ${pi/2}" xyz=".042 -0.098 0.22"/>
   </joint>
   <link name="vicon/marker4">
@@ -89,5 +89,5 @@
     <parent link="base"/>
     <child link="vicon/marker4"/>
-    <origin rpy="0 0 ${pi/2}" xyz="-0.101 0.059 0.370"/>
+    <origin rpy="0 0 ${pi/2}" xyz="-0.101 0.059 0.360"/>
   </joint>
   <link name="vicon/marker5">
@@ -109,5 +109,5 @@
     <parent link="base"/>
     <child link="vicon/marker5"/>
-    <origin rpy="0 0 ${pi/2}" xyz="-0.101 -0.059 0.370"/>
+    <origin rpy="0 0 ${pi/2}" xyz="-0.101 -0.059 0.360"/>
   </joint>
 </robot>
